File: hardware/eagle/usb-pedal.brd (EAGLE design)
At the start: 96.3 x 99.1 mm, 22 parts

Commit message: Add rev.1 board
Rev.1 solves the slight inconsistency of rev.0's microcontroller
board placement.
Now the board should be placed 'as you see it' while in the previous
version the silkscreen didn't actually match the correct board placement.
Parts:
- moved J4 17.0 mm to (63.5, 49.1)
- moved J3 17.0 mm to (80.5, 49.1)
- turned R1 to 0 degrees
- turned R2 to 0 degrees
- turned R3 to 0 degrees
Routing:
- net A1: track 133.7 -> 140.5 mm
- net A0: track 96.9 -> 90.6 mm, vias 0 -> 1
- net A2: track 141.7 -> 137.8 mm
Other:
- board text added: "USB Pedal rev. 1 Designed by Dimitris Platis http://plat.is/usb-pedal"
- board text removed: "USB Pedal rev. 0 Designed by Dimitris Platis http://plat.is/usb-pedal"
